File: kicad/ESP8266_FSBrowser.sch (KiCad schematic (older format))
At the start: 19 parts, among them P1 POWER, P2 ADC, P3 SERIAL, P4 GPIO, SW1 RESET, SW2 AP_ENABLE, SW3 FLASH, U1 ESP-12E, U2 LM1117-3.3

Commit message: Play with kicad files
Parts:
- removed P2: ADC, Pin_Headers:Pin_Header_Straight_1x02, symbol CONN_01X02
- removed U2: LM1117-3.3, TO_SOT_Packages_SMD:SOT-223, symbol LM1117-3.3
- added C3: 470p, Capacitors_SMD:C_0603, symbol C_Small
- added C4: 100u, Capacitors_SMD:c_elec_6.3x5.8, symbol CP1_Small
- added C5: 470p, Capacitors_SMD:C_0603, symbol C
- added R10: 0, Resistors_SMD:R_0603, symbol R
- added R11, R12: 470, Resistors_SMD:R_0603, symbol R
- added R13: 220k(1%), Resistors_SMD:R_0603, symbol R
- added R14: 100k(1%), Resistors_SMD:R_0603, symbol R
- added R8: 10k, Resistors_SMD:R_0603, symbol R
- added R9: 220, Resistors_SMD:R_0603, symbol R
- added U2: SPX3819M5-L-3-3, TO_SOT_Packages_SMD:SOT-23-5, symbol SPX3819M5-L-3-3
- C1: value 10u -> 1u; footprint Capacitors_Tantalum_SMD:TantalC_SizeU_EIA-6032 -> Capacitors_SMD:C_0603; symbol CP_Small -> C
- C2: value 1u -> 10u; footprint Capacitors_Tantalum_SMD:TantalC_SizeS_EIA-3216 -> Capacitors_SMD:C_0603; symbol CP_Small -> C
- P2: renamed from P4; footprint Pin_Headers:Pin_Header_Straight_2x06 -> Pin_Headers:Pin_Header_Straight_2x12; symbol CONN_02X06 -> CONN_02X12
- R5: value 330 -> 470
Connections:
- net +3V3: now also R2.2, R3.2, R4.2, R8.2, U2.5 (VOUT); no longer R2.1, R3.1, R4.1, R7.1
- net ADC: now also P2.22 (P22), R13.2, R14.1
- net GND: now also P2.13 (P13), P2.15 (P15), P2.17 (P17), P2.19 (P19), P2.21 (P21), P2.23 (P23), SW1.1, C3.2, C4.2, C5.2, R14.2, U2.2 (GND); no longer SW1.2
- net GPIO12: now also P2.10 (P10); no longer P2.6 (P6)
- net GPIO13: now also P2.8 (P8); no longer P2.4 (P4)
- net GPIO14: now also P2.6 (P6); no longer P2.2 (P2)
- net GPIO2: now also P2.16 (P16), R3.1; no longer P2.12 (P12), R4.2
- net GPIO5: now also P2.12 (P12); no longer P2.8 (P8)
- net RST: now also P2.20 (P20), C3.1, R10.1, R8.1; no longer R7.2, SW1.1, U1.4 (GPIO16)
- net GPIO15: now reaches R1.1, U1.16 (GPIO15)
- net at U1.21 (RXD): now also R12.2; no longer P3.3 (P3)
- net at U1.22 (TXD): now also R11.2; no longer P3.2 (P2)
- net CH_PD: now reaches U1.3 (CH_PD)
- net CH_PD: now also R2.1; no longer R2.2
- net +5V: now reaches C1.1, P1.2 (P2)
- net +5V: now also U2.1 (VIN), U2.3 (EN)
- net AP_EN renamed GPIO4
- net GPIO4: now also P2.14 (P14); no longer P2.10 (P10)
- new net: R9.1, SW3.1
- new net: R10.2, R7.2, SW1.2
- new net: P3.2 (P2), R11.1
- new net: P3.3 (P3), R12.1
- new net: C5.1, U2.4 (ADJ/BYP)
- new net ADC_EX: P2.24 (P24), R13.1
- new net GPIO0: P2.18 (P18), R4.1, R9.2, U1.18 (GPIO0)
- new net GPIO16: D1.1 (K), R7.1, U1.4 (GPIO16)
Other:
- moved on the sheet: D1, P1, R1, R2, R3, R4, R5, R6, R7, SW1, SW2, SW3

Commit message: Revert "Play with kicad files"
This reverts commit 04bb3029db1baf8c5355bf4588b1dad35f342a4f.
Parts:
- removed C3: 470p, Capacitors_SMD:C_0603, symbol C_Small
- removed C4: 100u, Capacitors_SMD:c_elec_6.3x5.8, symbol CP1_Small
- removed C5: 470p, Capacitors_SMD:C_0603, symbol C
- removed R10: 0, Resistors_SMD:R_0603, symbol R
- removed R11, R12: 470, Resistors_SMD:R_0603, symbol R
- removed R13: 220k(1%), Resistors_SMD:R_0603, symbol R
- removed R14: 100k(1%), Resistors_SMD:R_0603, symbol R
- removed R8: 10k, Resistors_SMD:R_0603, symbol R
- removed R9: 220, Resistors_SMD:R_0603, symbol R
- removed U2: SPX3819M5-L-3-3, TO_SOT_Packages_SMD:SOT-23-5, symbol SPX3819M5-L-3-3
- added P2: ADC, Pin_Headers:Pin_Header_Straight_1x02, symbol CONN_01X02
- added U2: LM1117-3.3, TO_SOT_Packages_SMD:SOT-223, symbol LM1117-3.3
- C1: value 1u -> 10u; footprint Capacitors_SMD:C_0603 -> Capacitors_Tantalum_SMD:TantalC_SizeU_EIA-6032; symbol C -> CP_Small
- C2: value 10u -> 1u; footprint Capacitors_SMD:C_0603 -> Capacitors_Tantalum_SMD:TantalC_SizeS_EIA-3216; symbol C -> CP_Small
- P4: renamed from P2; footprint Pin_Headers:Pin_Header_Straight_2x12 -> Pin_Headers:Pin_Header_Straight_2x06; symbol CONN_02X12 -> CONN_02X06
- R5: value 470 -> 330
Connections:
- net +3V3: now also R2.1, R3.1, R4.1, R7.1, U2.2 (VO), U2.4 (VO); no longer R2.2, R3.2, R4.2
- net ADC: now also P2.2 (P2); no longer P4.22 (P22)
- net GND: now also SW1.2, P2.1 (P1), U2.1 (GND/ADJ); no longer P4.13 (P13), P4.15 (P15), P4.17 (P17), P4.19 (P19), P4.21 (P21), P4.23 (P23), SW1.1
- net GPIO12: now also P4.6 (P6); no longer P4.10 (P10)
- net GPIO13: now also P4.4 (P4); no longer P4.8 (P8)
- net GPIO14: now also P4.2 (P2); no longer P4.6 (P6)
- net GPIO2: now also P4.12 (P12), R4.2; no longer P4.16 (P16), R3.1
- net GPIO5: now also P4.8 (P8); no longer P4.12 (P12)
- net RST: now also R7.2, SW1.1, U1.4 (GPIO16); no longer P4.20 (P20)
- net at U1.21 (RXD): now also P3.3 (P3)
- net at U1.22 (TXD): now also P3.2 (P2)
- net at SW3.1: now also D1.1 (K), R3.2, U1.18 (GPIO0)
- net +5V: no longer names the net of C1.1, P1.2 (P2)
- net +5V: now also U2.3 (VI)
- removed net ADC_EX: P4.24 (P24)
- net CH_PD: no longer names the net of U1.3 (CH_PD)
- net CH_PD: now also R2.2; no longer R2.1
- removed net GPIO0: P4.18 (P18), R4.1, U1.18 (GPIO0)
- net GPIO15: no longer names the net of R1.1, U1.16 (GPIO15)
- removed net GPIO16: D1.1 (K), R7.1, U1.4 (GPIO16)
- net GPIO4 renamed AP_EN
- net AP_EN: now also P4.10 (P10); no longer P4.14 (P14)
Other:
- moved on the sheet: D1, P1, R1, R2, R3, R4, R5, R6, R7, SW1, SW2, SW3
